Commit message: Add dual Piper teleop support with home position management
- Add read_piper_joints.py to read/save/restore dual arm home positions
- Add teleop_dual_piper_hardware.py for dual arm teleoperation
- Add dual_piper_teleop_controller.py and dual_piper.urdf
- Update piper_teleop_controller.py to load home_positions.json on startup and shutdown
- Fix shutdown to return arms to saved home position instead of hardcoded default

Co-Authored-By: Claude Sonnet 4.6 <noreply@anthropic.com>

File: XRoboToolkit-Teleop-Sample-Python/assets/gen72/dual_gen72.urdf (robot description, URDF)
Before this commit: robot dual_gen72, 17 links, 16 joints
Joints:
- joint world_to_left_base: origin xyz=0 0.3 0 rpy=0 0 0 -> xyz=0 0.3 0 rpy=0 0 3.14159
